Commit message: BDX-R URDF V2
Created new URDF facing x direction, split foot pads, and with covers.

File: BDX-R_description/BDX-R.urdf (robot description, URDF)
Before this commit: robot BDX-R, 23 links, 22 joints
Links:
- added link Antenna, mass 0.02; collision mesh filename=package://BDX-R_description/meshes/Antenna.stl scale=0.001 0.001 0.001; visual mesh filename=package://BDX-R_description/meshes/Antenna.stl scale=0.001 0.001 0.001
- added link AntennaBox, mass 0.065; collision mesh filename=package://BDX-R_description/meshes/AntennaBox.stl scale=0.001 0.001 0.001; visual mesh filename=package://BDX-R_description/meshes/AntennaBox.stl scale=0.001 0.001 0.001
- added link BackCover, mass 0.35; collision mesh filename=package://BDX-R_description/meshes/BackCover.stl scale=0.001 0.001 0.001; visual mesh filename=package://BDX-R_description/meshes/BackCover.stl scale=0.001 0.001 0.001
- added link BackFrame, mass 0.1; collision mesh filename=package://BDX-R_description/meshes/BackFrame.stl scale=0.001 0.001 0.001; visual mesh filename=package://BDX-R_description/meshes/BackFrame.stl scale=0.001 0.001 0.001
- added link BottomCover, mass 0.03; collision mesh filename=package://BDX-R_description/meshes/BottomCover.stl scale=0.001 0.001 0.001; visual mesh filename=package://BDX-R_description/meshes/BottomCover.stl scale=0.001 0.001 0.001
- added link FrontCover, mass 0.4; collision mesh filename=package://BDX-R_description/meshes/FrontCover.stl scale=0.001 0.001 0.001; visual mesh filename=package://BDX-R_description/meshes/FrontCover.stl scale=0.001 0.001 0.001
- added link LeftAnkleCover, mass 0.01; collision mesh filename=package://BDX-R_description/meshes/LeftAnkleCover.stl scale=0.001 0.001 0.001; visual mesh filename=package://BDX-R_description/meshes/LeftAnkleCover.stl scale=0.001 0.001 0.001
- added link LeftBottomLegCover, mass 0.1; collision mesh filename=package://BDX-R_description/meshes/LeftBottomLegCover.stl scale=0.001 0.001 0.001; visual mesh filename=package://BDX-R_description/meshes/LeftBottomLegCover.stl scale=0.001 0.001 0.001
- added link LeftFootCover, mass 0.01; collision mesh filename=package://BDX-R_description/meshes/LeftFootCover.stl scale=0.001 0.001 0.001; visual mesh filename=package://BDX-R_description/meshes/LeftFootCover.stl scale=0.001 0.001 0.001
- added link LeftFootPad, mass 0.05; collision mesh filename=package://BDX-R_description/meshes/LeftFootPad.stl scale=0.001 0.001 0.001; visual mesh filename=package://BDX-R_description/meshes/LeftFootPad.stl scale=0.001 0.001 0.001
- added link LeftLegBottomPlug, mass 0.01; collision mesh filename=package://BDX-R_description/meshes/LeftLegBottomPlug.stl scale=0.001 0.001 0.001; visual mesh filename=package://BDX-R_description/meshes/LeftLegBottomPlug.stl scale=0.001 0.001 0.001
- added link LeftLegUpperPlug, mass 0.01; collision mesh filename=package://BDX-R_description/meshes/LeftLegUpperPlug.stl scale=0.001 0.001 0.001; visual mesh filename=package://BDX-R_description/meshes/LeftLegUpperPlug.stl scale=0.001 0.001 0.001
- added link LeftUpperLegCover, mass 0.1; collision mesh filename=package://BDX-R_description/meshes/LeftUpperLegCover.stl scale=0.001 0.001 0.001; visual mesh filename=package://BDX-R_description/meshes/LeftUpperLegCover.stl scale=0.001 0.001 0.001
- added link RightAnkleCover, mass 0.02; collision mesh filename=package://BDX-R_description/meshes/RightAnkleCover.stl scale=0.001 0.001 0.001; visual mesh filename=package://BDX-R_description/meshes/RightAnkleCover.stl scale=0.001 0.001 0.001
- added link RightBottomLegCover, mass 0.1; collision mesh filename=package://BDX-R_description/meshes/RightBottomLegCover.stl scale=0.001 0.001 0.001; visual mesh filename=package://BDX-R_description/meshes/RightBottomLegCover.stl scale=0.001 0.001 0.001
- added link RightFootCover, mass 0.02; collision mesh filename=package://BDX-R_description/meshes/RightFootCover.stl scale=0.001 0.001 0.001; visual mesh filename=package://BDX-R_description/meshes/RightFootCover.stl scale=0.001 0.001 0.001
- added link RightFootPad, mass 0.05; collision mesh filename=package://BDX-R_description/meshes/RightFootPad.stl scale=0.001 0.001 0.001; visual mesh filename=package://BDX-R_description/meshes/RightFootPad.stl scale=0.001 0.001 0.001
- added link RightLegBottomPlug, mass 0.01; collision mesh filename=package://BDX-R_description/meshes/RightLegBottomPlug.stl scale=0.001 0.001 0.001; visual mesh filename=package://BDX-R_description/meshes/RightLegBottomPlug.stl scale=0.001 0.001 0.001
- added link RightLegUpperPlug, mass 0.01; collision mesh filename=package://BDX-R_description/meshes/RightLegUpperPlug.stl scale=0.001 0.001 0.001; visual mesh filename=package://BDX-R_description/meshes/RightLegUpperPlug.stl scale=0.001 0.001 0.001
- added link RightUpperLegCover, mass 0.1; collision mesh filename=package://BDX-R_description/meshes/RightUpperLegCover.stl scale=0.001 0.001 0.001; visual mesh filename=package://BDX-R_description/meshes/RightUpperLegCover.stl scale=0.001 0.001 0.001
- added link TopLeftCover, mass 0.1; collision mesh filename=package://BDX-R_description/meshes/TopLeftCover.stl scale=0.001 0.001 0.001; visual mesh filename=package://BDX-R_description/meshes/TopLeftCover.stl scale=0.001 0.001 0.001
- added link TopRightCover, mass 0.1; collision mesh filename=package://BDX-R_description/meshes/TopRightCover.stl scale=0.001 0.001 0.001; visual mesh filename=package://BDX-R_description/meshes/TopRightCover.stl scale=0.001 0.001 0.001
- link Battery: mass 1.0730942884373287 -> 1.00; geometry collision mesh filename=package://BDX-R_description/meshes/Battery.stl scale=0.001 0.001 0.001; visual mesh filename=package://BDX-R_description/meshes/Battery.stl scale=0.001 0.001 0.001
- link IMU_Mount: mass 0.01915492960248384 -> 0.02; geometry collision mesh filename=package://BDX-R_description/meshes/IMU_Mount.stl scale=0.001 0.001 0.001; visual mesh filename=package://BDX-R_description/meshes/IMU_Mount.stl scale=0.001 0.001 0.001
- link Jetson_Mount: mass 0.24846958841683578 -> 0.3; geometry collision mesh filename=package://BDX-R_description/meshes/Jetson_Mount.stl scale=0.001 0.001 0.001; visual mesh filename=package://BDX-R_description/meshes/Jetson_Mount.stl scale=0.001 0.001 0.001
- link Left_Ankle_Motor: geometry collision mesh filename=package://BDX-R_description/meshes/Left_Ankle_Motor.stl scale=0.001 0.001 0.001; visual mesh filename=package://BDX-R_description/meshes/Left_Ankle_Motor.stl scale=0.001 0.001 0.001
- link Left_Foot: mass 0.3335675718817209 -> 0.22236469248575175; geometry collision mesh filename=package://BDX-R_description/meshes/Left_Foot.stl scale=0.001 0.001 0.001; visual mesh filename=package://BDX-R_description/meshes/Left_Foot.stl scale=0.001 0.001 0.001
- link Left_Hip_Connector: geometry collision mesh filename=package://BDX-R_description/meshes/Left_Hip_Connector.stl scale=0.001 0.001 0.001; visual mesh filename=package://BDX-R_description/meshes/Left_Hip_Connector.stl scale=0.001 0.001 0.001
- link Left_Hip_Pitch_Motor: geometry collision mesh filename=package://BDX-R_description/meshes/Left_Hip_Pitch_Motor.stl scale=0.001 0.001 0.001; visual mesh filename=package://BDX-R_description/meshes/Left_Hip_Pitch_Motor.stl scale=0.001 0.001 0.001
- link Left_Hip_Roll_Motor: geometry collision mesh filename=package://BDX-R_description/meshes/Left_Hip_Roll_Motor.stl scale=0.001 0.001 0.001; visual mesh filename=package://BDX-R_description/meshes/Left_Hip_Roll_Motor.stl scale=0.001 0.001 0.001
- link Left_Hip_Yaw_Motor: geometry collision mesh filename=package://BDX-R_description/meshes/Left_Hip_Yaw_Motor.stl scale=0.001 0.001 0.001; visual mesh filename=package://BDX-R_description/meshes/Left_Hip_Yaw_Motor.stl scale=0.001 0.001 0.001
- link Left_Knee_Motor: geometry collision mesh filename=package://BDX-R_description/meshes/Left_Knee_Motor.stl scale=0.001 0.001 0.001; visual mesh filename=package://BDX-R_description/meshes/Left_Knee_Motor.stl scale=0.001 0.001 0.001
- link Left_Lower_Leg: mass 0.38681765132349716 -> 0.4; geometry collision mesh filename=package://BDX-R_description/meshes/Left_Lower_Leg.stl scale=0.001 0.001 0.001; visual mesh filename=package://BDX-R_description/meshes/Left_Lower_Leg.stl scale=0.001 0.001 0.001
- link Left_Upper_Leg: geometry collision mesh filename=package://BDX-R_description/meshes/Left_Upper_Leg.stl scale=0.001 0.001 0.001; visual mesh filename=package://BDX-R_description/meshes/Left_Upper_Leg.stl scale=0.001 0.001 0.001
- link Neck_Motor: mass 0.910452277662412 -> 0.9104522776624081; geometry collision mesh filename=package://BDX-R_description/meshes/Neck_Motor.stl scale=0.001 0.001 0.001; visual mesh filename=package://BDX-R_description/meshes/Neck_Motor.stl scale=0.001 0.001 0.001
- link Right_Ankle_Motor: mass 0.36575911696028485 -> 0.3657591169602799; geometry collision mesh filename=package://BDX-R_description/meshes/Right_Ankle_Motor.stl scale=0.001 0.001 0.001; visual mesh filename=package://BDX-R_description/meshes/Right_Ankle_Motor.stl scale=0.001 0.001 0.001
- link Right_Foot: mass 0.3335675718740702 -> 0.2223646924781009; geometry collision mesh filename=package://BDX-R_description/meshes/Right_Foot.stl scale=0.001 0.001 0.001; visual mesh filename=package://BDX-R_description/meshes/Right_Foot.stl scale=0.001 0.001 0.001
- link Right_Hip_Connector: geometry collision mesh filename=package://BDX-R_description/meshes/Right_Hip_Connector.stl scale=0.001 0.001 0.001; visual mesh filename=package://BDX-R_description/meshes/Right_Hip_Connector.stl scale=0.001 0.001 0.001
- link Right_Hip_Pitch_Motor: geometry collision mesh filename=package://BDX-R_description/meshes/Right_Hip_Pitch_Motor.stl scale=0.001 0.001 0.001; visual mesh filename=package://BDX-R_description/meshes/Right_Hip_Pitch_Motor.stl scale=0.001 0.001 0.001
- link Right_Hip_Roll_Motor: geometry collision mesh filename=package://BDX-R_description/meshes/Right_Hip_Roll_Motor.stl scale=0.001 0.001 0.001; visual mesh filename=package://BDX-R_description/meshes/Right_Hip_Roll_Motor.stl scale=0.001 0.001 0.001
- link Right_Hip_Yaw_Motor: geometry collision mesh filename=package://BDX-R_description/meshes/Right_Hip_Yaw_Motor.stl scale=0.001 0.001 0.001; visual mesh filename=package://BDX-R_description/meshes/Right_Hip_Yaw_Motor.stl scale=0.001 0.001 0.001
- link Right_Knee_Motor: mass 0.9104522723338447 -> 0.9104522723338422; geometry collision mesh filename=package://BDX-R_description/meshes/Right_Knee_Motor.stl scale=0.001 0.001 0.001; visual mesh filename=package://BDX-R_description/meshes/Right_Knee_Motor.stl scale=0.001 0.001 0.001
- link Right_Lower_Leg: mass 0.3868176513234967 -> 0.4; geometry collision mesh filename=package://BDX-R_description/meshes/Right_Lower_Leg.stl scale=0.001 0.001 0.001; visual mesh filename=package://BDX-R_description/meshes/Right_Lower_Leg.stl scale=0.001 0.001 0.001
- link Right_Upper_Leg: geometry collision mesh filename=package://BDX-R_description/meshes/Right_Upper_Leg.stl scale=0.001 0.001 0.001; visual mesh filename=package://BDX-R_description/meshes/Right_Upper_Leg.stl scale=0.001 0.001 0.001
- link base_link: mass 1.9551413921032492 -> 1.6; geometry collision mesh filename=package://BDX-R_description/meshes/base_link.stl scale=0.001 0.001 0.001; visual mesh filename=package://BDX-R_description/meshes/base_link.stl scale=0.001 0.001 0.001
Joints:
- removed joint Rigid 18
- removed joint Rigid 20
- removed joint Rigid 25
- removed joint Rigid 32
- added joint Rigid 1: type fixed, parent base_link, child Right_Hip_Yaw_Motor, origin xyz=0.019472 0.018451 0.046444 rpy=0 0 0
- added joint Rigid 10: type fixed, parent base_link, child Jetson_Mount, origin xyz=0.076306 0.077202 0.016701 rpy=0 0 0
- added joint Rigid 11: type fixed, parent base_link, child Neck_Motor, origin xyz=0.076005 0.108952 0.134165 rpy=0 0 0
- added joint Rigid 12: type fixed, parent base_link, child Battery, origin xyz=0.0 -0.002881 0.093743 rpy=0 0 0
- added joint Rigid 13: type fixed, parent BackCover, child Antenna, origin xyz=-0.019105 0.0 -6e-06 rpy=0 0 0
- added joint Rigid 19: type fixed, parent Right_Hip_Pitch_Motor, child Right_Upper_Leg, origin xyz=0.018686 -0.0025 0.045297 rpy=0 0 0
- added joint Rigid 2: type fixed, parent base_link, child Left_Hip_Yaw_Motor, origin xyz=0.019472 0.155954 0.046444 rpy=0 0 0
- added joint Rigid 21: type fixed, parent Right_Upper_Leg, child Right_Knee_Motor, origin xyz=-0.052447 0.0 -0.104765 rpy=0 0 0
- added joint Rigid 29: type fixed, parent Right_Upper_Leg, child RightUpperLegCover, origin xyz=-0.008513 -0.0465 0.000589 rpy=0 0 0
- added joint Rigid 3: type fixed, parent base_link, child BottomCover, origin xyz=0.002222 0.024202 -0.1018 rpy=0 0 0
- added joint Rigid 30: type fixed, parent RightUpperLegCover, child RightLegUpperPlug, origin xyz=-0.006969 -0.02025 -0.047727 rpy=0 0 0
- added joint Rigid 31: type fixed, parent RightBottomLegCover, child RightLegBottomPlug, origin xyz=0.06601 -0.02025 -0.009329 rpy=0 0 0
- added joint Rigid 36: type fixed, parent Left_Lower_Leg, child Left_Ankle_Motor, origin xyz=0.044852 -0.00934 -0.093516 rpy=0 0 0
- added joint Rigid 38: type fixed, parent Left_Foot, child LeftFootPad, origin xyz=0.026824 -0.018025 -0.059089 rpy=0 0 0
- added joint Rigid 39: type fixed, parent Left_Foot, child LeftFootCover, origin xyz=-0.041648 0.0105 -0.042644 rpy=0 0 0
- added joint Rigid 4: type fixed, parent base_link, child BackFrame, origin xyz=-0.096859 0.137077 0.060614 rpy=0 0 0
- added joint Rigid 40: type fixed, parent Left_Lower_Leg, child LeftAnkleCover, origin xyz=0.018114 -0.045377 -0.162552 rpy=0 0 0
- added joint Rigid 41: type fixed, parent Left_Upper_Leg, child LeftBottomLegCover, origin xyz=-0.106078 0.0465 -0.112095 rpy=0 0 0
- added joint Rigid 42: type fixed, parent Left_Upper_Leg, child LeftUpperLegCover, origin xyz=0.028989 0.0465 0.000643 rpy=0 0 0
- added joint Rigid 43: type fixed, parent LeftBottomLegCover, child LeftLegBottomPlug, origin xyz=0.06601 0.02025 -0.009329 rpy=0 0 0
- added joint Rigid 44: type fixed, parent LeftUpperLegCover, child LeftLegUpperPlug, origin xyz=-0.013452 0.02025 -0.033648 rpy=0 0 0
- added joint Rigid 5: type fixed, parent BackFrame, child BackCover, origin xyz=-0.066834 6.8e-05 -0.029977 rpy=0 0 0
- added joint Rigid 6: type fixed, parent base_link, child FrontCover, origin xyz=0.071231 -0.015041 0.058018 rpy=0 0 0
- added joint Rigid 7: type fixed, parent base_link, child TopLeftCover, origin xyz=-0.068283 0.178249 0.108311 rpy=0 0 0
- added joint Rigid 8: type fixed, parent base_link, child TopRightCover, origin xyz=-0.068283 -0.003845 0.108311 rpy=0 0 0
- added joint Rigid 9: type fixed, parent base_link, child IMU_Mount, origin xyz=-0.047178 0.066302 0.110944 rpy=0 0 0
- joint Left_Ankle: axis -1.0 0.0 -0.0 -> -0.0 -1.0 -0.0; limit lower=-0.85 upper=1.3 effort=17 velocity=40 -> lower=-0.85 upper=1.3 effort=11.9 velocity=37.699; origin xyz=0.004 0.0 0.0 rpy=0 0 0 -> xyz=0.00052 0.004 -0.036497 rpy=0 0 0
- joint Left_Hip_Pitch: axis 1.0 0.0 0.0 -> -0.0 -1.0 0.0; limit lower=-0.5 upper=1 effort=60 velocity=20 -> lower=-0.5 upper=1 effort=42 velocity=18.849; origin xyz=0.07125 0.008647 0.001341 rpy=0 0 0 -> xyz=-0.008647 0.07125 0.001341 rpy=0 0 0
- joint Left_Hip_Roll: axis 0.0 1.0 0.0 -> 1.0 -0.0 0.0; limit lower=-0.3 upper=0.3 effort=60 velocity=20 -> lower=-0.3 upper=0.3 effort=42 velocity=18.849; origin xyz=0.0125 -0.018 -0.064284 rpy=0 0 0 -> xyz=0.018 0.0125 -0.064284 rpy=0 0 0
- joint Left_Hip_Yaw: limit lower=-0.35 upper=0.5 effort=60 velocity=20 -> lower=-0.5 upper=0.35 effort=42 velocity=18.849; origin xyz=-0.018751 -0.04527 -0.0025 rpy=0 0 0 -> xyz=-0.04527 -0.018752 -0.0025 rpy=0 0 0
- joint Left_Knee: axis 1.0 0.0 0.0 -> -0.0 -1.0 0.0; limit lower=-0.95 upper=1.2 effort=60 velocity=20 -> lower=-0.95 upper=1.2 effort=42.0 velocity=18.849; origin xyz=-0.0025 0.0 0.0 rpy=0 0 0 -> xyz=-0.019146 -0.042 -0.045104 rpy=0 0 0
- joint Right_Ankle: axis 1.0 -0.0 0.0 -> 0.0 -1.0 0.0; limit lower=-1.3 upper=0.85 effort=17 velocity=40 -> lower=-1.3 upper=0.85 effort=11.9 velocity=37.699; origin xyz=-0.004 0.0 0.0 rpy=0 0 0 -> xyz=0.023858 -0.004 -0.027623 rpy=0 0 0
- joint Right_Hip_Pitch: axis -1.0 -0.0 -0.0 -> -0.0 -1.0 -0.0; limit lower=-1 upper=0.5 effort=60 velocity=20 -> lower=-1 upper=0.5 effort=42 velocity=18.849; origin xyz=-0.07125 0.008647 0.001341 rpy=0 0 0 -> xyz=-0.008647 -0.07125 0.001341 rpy=0 0 0
- joint Right_Hip_Roll: axis -0.0 1.0 0.0 -> -1.0 0.0 -0.0; limit lower=-0.3 upper=0.3 effort=60 velocity=20 -> lower=-0.3 upper=0.3 effort=42 velocity=18.849; origin xyz=-0.0125 -0.018 -0.064284 rpy=0 0 0 -> xyz=0.018 -0.0125 -0.064284 rpy=0 0 0
- joint Right_Hip_Yaw: axis -0.0 0.0 1.0 -> 0.0 0.0 1.0; limit lower=-0.5 upper=0.35 effort=60 velocity=20 -> lower=-0.5 upper=0.35 effort=42 velocity=18.849; origin xyz=0.018751 -0.04527 -0.0025 rpy=0 0 0 -> xyz=-0.04527 0.018751 -0.0025 rpy=0 0 0
- joint Right_Knee: axis -1.0 -0.0 -0.0 -> -0.0 -1.0 -0.0; limit lower=-1.2 upper=0.95 effort=60 velocity=20 -> lower=-1.2 upper=0.95 effort=42 velocity=18.849; origin xyz=0.0025 0.0 0.0 rpy=0 0 0 -> xyz=-0.045432 0.0025 -0.018355 rpy=0 0 0
- joint Rigid 14: child Right_Hip_Yaw_Motor -> AntennaBox; origin xyz=-0.068751 0.15827 0.046444 rpy=0 0 0 -> xyz=-0.008 0.0 0.0 rpy=0 0 0; parent base_link -> Antenna
- joint Rigid 23: origin xyz=0.00934 -0.045337 -0.130013 rpy=0 0 0 -> xyz=0.021506 0.00934 -0.102367 rpy=0 0 0
- joint Rigid 24: child IMU_Mount -> RightAnkleCover; origin xyz=-0.0209 0.14962 0.110944 rpy=0 0 0 -> xyz=0.07256 0.045378 -0.097474 rpy=0 0 0; parent base_link -> Right_Lower_Leg
- joint Rigid 26: child Jetson_Mount -> RightFootPad; origin xyz=-0.01 0.010896 0.016701 rpy=0 0 0 -> xyz=0.026823 0.018026 -0.059089 rpy=0 0 0; parent base_link -> Right_Foot
- joint Rigid 27: child Neck_Motor -> RightFootCover; origin xyz=0.02175 -0.001404 0.044506 rpy=0 0 0 -> xyz=-0.041649 -0.0105 -0.042645 rpy=0 0 0; parent base_link -> Right_Foot
- joint Rigid 28: child Left_Hip_Yaw_Motor -> RightBottomLegCover; origin xyz=0.068751 0.15827 0.046444 rpy=0 0 0 -> xyz=-0.14358 -0.0465 -0.112149 rpy=0 0 0; parent base_link -> Right_Upper_Leg
- joint Rigid 33: child Left_Knee_Motor -> Left_Upper_Leg; origin xyz=0.0 0.097879 -0.12312 rpy=0 0 0 -> xyz=-0.018816 0.0025 0.045243 rpy=0 0 0; parent Left_Upper_Leg -> Left_Hip_Pitch_Motor
- joint Rigid 34: child Left_Ankle_Motor -> Left_Knee_Motor; origin xyz=-0.00934 -0.045337 -0.130013 rpy=0 0 0 -> xyz=-0.041231 0.0392 -0.077962 rpy=0 0 0; parent Left_Lower_Leg -> Left_Upper_Leg
