Commit message: cleans description and repo

File: BDX-R-Description/BDX-R.urdf (robot description, URDF)
Before this commit: robot BDX-R, 45 links, 44 joints
Links:
- link Antenna: geometry collision mesh filename=package://BDX-R-Description/meshes/Antenna.stl scale=0.001 0.001 0.001; visual mesh filename=package://BDX-R-Description/meshes/Antenna.stl scale=0.001 0.001 0.001
- link AntennaBox: geometry collision mesh filename=package://BDX-R-Description/meshes/AntennaBox.stl scale=0.001 0.001 0.001; visual mesh filename=package://BDX-R-Description/meshes/AntennaBox.stl scale=0.001 0.001 0.001
- link BackCover: geometry collision mesh filename=package://BDX-R-Description/meshes/BackCover.stl scale=0.001 0.001 0.001; visual mesh filename=package://BDX-R-Description/meshes/BackCover.stl scale=0.001 0.001 0.001
- link BackFrame: geometry collision mesh filename=package://BDX-R-Description/meshes/BackFrame.stl scale=0.001 0.001 0.001; visual mesh filename=package://BDX-R-Description/meshes/BackFrame.stl scale=0.001 0.001 0.001
- link Battery: geometry collision mesh filename=package://BDX-R-Description/meshes/Battery.stl scale=0.001 0.001 0.001; visual mesh filename=package://BDX-R-Description/meshes/Battery.stl scale=0.001 0.001 0.001
- link BottomCover: geometry collision mesh filename=package://BDX-R-Description/meshes/BottomCover.stl scale=0.001 0.001 0.001; visual mesh filename=package://BDX-R-Description/meshes/BottomCover.stl scale=0.001 0.001 0.001
- link FrontCover: geometry collision mesh filename=package://BDX-R-Description/meshes/FrontCover.stl scale=0.001 0.001 0.001; visual mesh filename=package://BDX-R-Description/meshes/FrontCover.stl scale=0.001 0.001 0.001
- link IMU_Mount: geometry collision mesh filename=package://BDX-R-Description/meshes/IMU_Mount.stl scale=0.001 0.001 0.001; visual mesh filename=package://BDX-R-Description/meshes/IMU_Mount.stl scale=0.001 0.001 0.001
- link Jetson_Mount: geometry collision mesh filename=package://BDX-R-Description/meshes/Jetson_Mount.stl scale=0.001 0.001 0.001; visual mesh filename=package://BDX-R-Description/meshes/Jetson_Mount.stl scale=0.001 0.001 0.001
- link LeftAnkleCover: geometry collision mesh filename=package://BDX-R-Description/meshes/LeftAnkleCover.stl scale=0.001 0.001 0.001; visual mesh filename=package://BDX-R-Description/meshes/LeftAnkleCover.stl scale=0.001 0.001 0.001
- link LeftBottomLegCover: geometry collision mesh filename=package://BDX-R-Description/meshes/LeftBottomLegCover.stl scale=0.001 0.001 0.001; visual mesh filename=package://BDX-R-Description/meshes/LeftBottomLegCover.stl scale=0.001 0.001 0.001
- link LeftFootCover: geometry collision mesh filename=package://BDX-R-Description/meshes/LeftFootCover.stl scale=0.001 0.001 0.001; visual mesh filename=package://BDX-R-Description/meshes/LeftFootCover.stl scale=0.001 0.001 0.001
- link LeftFootPad: geometry collision mesh filename=package://BDX-R-Description/meshes/LeftFootPad.stl scale=0.001 0.001 0.001; visual mesh filename=package://BDX-R-Description/meshes/LeftFootPad.stl scale=0.001 0.001 0.001
- link LeftLegBottomPlug: geometry collision mesh filename=package://BDX-R-Description/meshes/LeftLegBottomPlug.stl scale=0.001 0.001 0.001; visual mesh filename=package://BDX-R-Description/meshes/LeftLegBottomPlug.stl scale=0.001 0.001 0.001
- link LeftLegUpperPlug: geometry collision mesh filename=package://BDX-R-Description/meshes/LeftLegUpperPlug.stl scale=0.001 0.001 0.001; visual mesh filename=package://BDX-R-Description/meshes/LeftLegUpperPlug.stl scale=0.001 0.001 0.001
- link LeftUpperLegCover: geometry collision mesh filename=package://BDX-R-Description/meshes/LeftUpperLegCover.stl scale=0.001 0.001 0.001; visual mesh filename=package://BDX-R-Description/meshes/LeftUpperLegCover.stl scale=0.001 0.001 0.001
- link Left_Ankle_Motor: geometry collision mesh filename=package://BDX-R-Description/meshes/Left_Ankle_Motor.stl scale=0.001 0.001 0.001; visual mesh filename=package://BDX-R-Description/meshes/Left_Ankle_Motor.stl scale=0.001 0.001 0.001
- link Left_Foot: geometry collision mesh filename=package://BDX-R-Description/meshes/Left_Foot.stl scale=0.001 0.001 0.001; visual mesh filename=package://BDX-R-Description/meshes/Left_Foot.stl scale=0.001 0.001 0.001
- link Left_Hip_Connector: geometry collision mesh filename=package://BDX-R-Description/meshes/Left_Hip_Connector.stl scale=0.001 0.001 0.001; visual mesh filename=package://BDX-R-Description/meshes/Left_Hip_Connector.stl scale=0.001 0.001 0.001
- link Left_Hip_Pitch_Motor: geometry collision mesh filename=package://BDX-R-Description/meshes/Left_Hip_Pitch_Motor.stl scale=0.001 0.001 0.001; visual mesh filename=package://BDX-R-Description/meshes/Left_Hip_Pitch_Motor.stl scale=0.001 0.001 0.001
- link Left_Hip_Roll_Motor: geometry collision mesh filename=package://BDX-R-Description/meshes/Left_Hip_Roll_Motor.stl scale=0.001 0.001 0.001; visual mesh filename=package://BDX-R-Description/meshes/Left_Hip_Roll_Motor.stl scale=0.001 0.001 0.001
- link Left_Hip_Yaw_Motor: geometry collision mesh filename=package://BDX-R-Description/meshes/Left_Hip_Yaw_Motor.stl scale=0.001 0.001 0.001; visual mesh filename=package://BDX-R-Description/meshes/Left_Hip_Yaw_Motor.stl scale=0.001 0.001 0.001
- link Left_Knee_Motor: geometry collision mesh filename=package://BDX-R-Description/meshes/Left_Knee_Motor.stl scale=0.001 0.001 0.001; visual mesh filename=package://BDX-R-Description/meshes/Left_Knee_Motor.stl scale=0.001 0.001 0.001
- link Left_Lower_Leg: geometry collision mesh filename=package://BDX-R-Description/meshes/Left_Lower_Leg.stl scale=0.001 0.001 0.001; visual mesh filename=package://BDX-R-Description/meshes/Left_Lower_Leg.stl scale=0.001 0.001 0.001
- link Left_Upper_Leg: geometry collision mesh filename=package://BDX-R-Description/meshes/Left_Upper_Leg.stl scale=0.001 0.001 0.001; visual mesh filename=package://BDX-R-Description/meshes/Left_Upper_Leg.stl scale=0.001 0.001 0.001
- link Neck_Motor: geometry collision mesh filename=package://BDX-R-Description/meshes/Neck_Motor.stl scale=0.001 0.001 0.001; visual mesh filename=package://BDX-R-Description/meshes/Neck_Motor.stl scale=0.001 0.001 0.001
- link RightAnkleCover: geometry collision mesh filename=package://BDX-R-Description/meshes/RightAnkleCover.stl scale=0.001 0.001 0.001; visual mesh filename=package://BDX-R-Description/meshes/RightAnkleCover.stl scale=0.001 0.001 0.001
- link RightBottomLegCover: geometry collision mesh filename=package://BDX-R-Description/meshes/RightBottomLegCover.stl scale=0.001 0.001 0.001; visual mesh filename=package://BDX-R-Description/meshes/RightBottomLegCover.stl scale=0.001 0.001 0.001
- link RightFootCover: geometry collision mesh filename=package://BDX-R-Description/meshes/RightFootCover.stl scale=0.001 0.001 0.001; visual mesh filename=package://BDX-R-Description/meshes/RightFootCover.stl scale=0.001 0.001 0.001
- link RightFootPad: geometry collision mesh filename=package://BDX-R-Description/meshes/RightFootPad.stl scale=0.001 0.001 0.001; visual mesh filename=package://BDX-R-Description/meshes/RightFootPad.stl scale=0.001 0.001 0.001
- link RightLegBottomPlug: geometry collision mesh filename=package://BDX-R-Description/meshes/RightLegBottomPlug.stl scale=0.001 0.001 0.001; visual mesh filename=package://BDX-R-Description/meshes/RightLegBottomPlug.stl scale=0.001 0.001 0.001
- link RightLegUpperPlug: geometry collision mesh filename=package://BDX-R-Description/meshes/RightLegUpperPlug.stl scale=0.001 0.001 0.001; visual mesh filename=package://BDX-R-Description/meshes/RightLegUpperPlug.stl scale=0.001 0.001 0.001
- link RightUpperLegCover: geometry collision mesh filename=package://BDX-R-Description/meshes/RightUpperLegCover.stl scale=0.001 0.001 0.001; visual mesh filename=package://BDX-R-Description/meshes/RightUpperLegCover.stl scale=0.001 0.001 0.001
- link Right_Ankle_Motor: geometry collision mesh filename=package://BDX-R-Description/meshes/Right_Ankle_Motor.stl scale=0.001 0.001 0.001; visual mesh filename=package://BDX-R-Description/meshes/Right_Ankle_Motor.stl scale=0.001 0.001 0.001
- link Right_Foot: geometry collision mesh filename=package://BDX-R-Description/meshes/Right_Foot.stl scale=0.001 0.001 0.001; visual mesh filename=package://BDX-R-Description/meshes/Right_Foot.stl scale=0.001 0.001 0.001
- link Right_Hip_Connector: geometry collision mesh filename=package://BDX-R-Description/meshes/Right_Hip_Connector.stl scale=0.001 0.001 0.001; visual mesh filename=package://BDX-R-Description/meshes/Right_Hip_Connector.stl scale=0.001 0.001 0.001
- link Right_Hip_Pitch_Motor: geometry collision mesh filename=package://BDX-R-Description/meshes/Right_Hip_Pitch_Motor.stl scale=0.001 0.001 0.001; visual mesh filename=package://BDX-R-Description/meshes/Right_Hip_Pitch_Motor.stl scale=0.001 0.001 0.001
- link Right_Hip_Roll_Motor: geometry collision mesh filename=package://BDX-R-Description/meshes/Right_Hip_Roll_Motor.stl scale=0.001 0.001 0.001; visual mesh filename=package://BDX-R-Description/meshes/Right_Hip_Roll_Motor.stl scale=0.001 0.001 0.001
- link Right_Hip_Yaw_Motor: geometry collision mesh filename=package://BDX-R-Description/meshes/Right_Hip_Yaw_Motor.stl scale=0.001 0.001 0.001; visual mesh filename=package://BDX-R-Description/meshes/Right_Hip_Yaw_Motor.stl scale=0.001 0.001 0.001
- link Right_Knee_Motor: geometry collision mesh filename=package://BDX-R-Description/meshes/Right_Knee_Motor.stl scale=0.001 0.001 0.001; visual mesh filename=package://BDX-R-Description/meshes/Right_Knee_Motor.stl scale=0.001 0.001 0.001
- link Right_Lower_Leg: geometry collision mesh filename=package://BDX-R-Description/meshes/Right_Lower_Leg.stl scale=0.001 0.001 0.001; visual mesh filename=package://BDX-R-Description/meshes/Right_Lower_Leg.stl scale=0.001 0.001 0.001
- link Right_Upper_Leg: geometry collision mesh filename=package://BDX-R-Description/meshes/Right_Upper_Leg.stl scale=0.001 0.001 0.001; visual mesh filename=package://BDX-R-Description/meshes/Right_Upper_Leg.stl scale=0.001 0.001 0.001
- link TopLeftCover: geometry collision mesh filename=package://BDX-R-Description/meshes/TopLeftCover.stl scale=0.001 0.001 0.001; visual mesh filename=package://BDX-R-Description/meshes/TopLeftCover.stl scale=0.001 0.001 0.001
- link TopRightCover: geometry collision mesh filename=package://BDX-R-Description/meshes/TopRightCover.stl scale=0.001 0.001 0.001; visual mesh filename=package://BDX-R-Description/meshes/TopRightCover.stl scale=0.001 0.001 0.001
- link base_link: geometry collision mesh filename=package://BDX-R-Description/meshes/base_link.stl scale=0.001 0.001 0.001; visual mesh filename=package://BDX-R-Description/meshes/base_link.stl scale=0.001 0.001 0.001
