Commit message: Add files via upload

File: BDX-R-Description/urdf/URDF.urdf (robot description, URDF)
Before this commit: robot URDF, 77 links, 76 joints
Links:
- removed link Right_Lower_leg-Cover
- added link Right_Lower_Leg_Cover, mass 0.36564522610609057; collision mesh filename=package://URDF_description/meshes/Right_Lower_Leg_Cover.stl scale=0.001 0.001 0.001; visual mesh filename=package://URDF_description/meshes/Right_Lower_Leg_Cover.stl scale=0.001 0.001 0.001
Joints:
- joint Rigid 73: child Right_Lower_leg-Cover -> Right_Lower_Leg_Cover

Commit message: Updated URDF for head and proper weights

File: BDX-R-Description/urdf/URDF.urdf (robot description, URDF)
Before this commit: robot URDF, 77 links, 76 joints
Links:
- link Back_Support: mass 1.4345660747046487 -> 0.1
- link Base_Top_Clamp: mass 0.34279762697415633 -> 0.044
- link Battery: mass 7.946971853050029 -> 1.25
- link Battery_Holder: mass 1.2003975073649495 -> 0.18
- link Bottom_Cover: mass 0.2325777541774406 -> 0.1
- link Camera_Mount: mass 0.23780328755101082 -> 0.04
- link Face: mass 0.3825323982770003 -> 0.1
- link Front_Cover: mass 3.016585112031044 -> 0.2
- link Front_Grill: mass 0.12278343435530116 -> 0.01
- link Front_Support: mass 1.3644492060488889 -> 0.15
- link Head_Base_Plate: mass 0.7026538517747032 -> 0.24
- link Head_Pitch_Motor_Support: mass 0.3978591096412742 -> 0.08
- link Head_Rear_Cover: mass 2.1083250067116728 -> 0.1
- link Head_Roll_Connector: mass 0.1909286096033978 -> 0.05
- link Head_Roll_Motor_Mount: mass 0.42782888507946565 -> 0.08
- link Left_Ankle_Cover: mass 0.10517582367621381 -> 0.01
- link Left_Cable_Support: mass 0.4093453218387253 -> 0.08
- link Left_Ear: mass 0.08364465059570073 -> 0.01
- link Left_Eye: mass 0.1126202923319544 -> 0.02
- link Left_Foot: mass 1.8791037125473142 -> 0.22
- link Left_Foot_Cover: mass 0.2778877451208695 -> 0.02
- link Left_Foot_Pad: mass 0.8235307524446849 -> 0.08
- link Left_Front_Cover: mass 0.5492461618694918 -> 0.1
- link Left_Head_Support: mass 0.15134820623495676 -> 0.04
- link Left_Hip_Bottom_Holder: mass 0.44482107671145055 -> 0.075
- link Left_Hip_Pitch_Motor: mass 0.880 -> 0.920
- link Left_Hip_Roll_Connector: mass 0.28535022457844034 -> 0.1
- link Left_Hip_Roll_Motor: mass 0.880 -> 0.920
- link Left_Hip_Top_Holder: mass 0.6080984706410992 -> 0.08
- link Left_Hip_Yaw_Motor: mass 0.880 -> 0.920
- link Left_Hip_Yaw_Support: mass 0.8129334554771345 -> 0.08
- link Left_Holder: mass 0.37776469464112955 -> 0.08
- link Left_Knee_Motor: mass 0.880 -> 0.920
- link Left_Lower_Leg: mass 2.8649012995453993 -> 0.33
- link Left_Lower_Leg_Cover: mass 0.6798560279056552 -> 0.057
- link Left_Top_Cover: mass 0.30626446288176407 -> 0.03
- link Left_Upper_Leg: mass 4.1882983071068365 -> 0.5
- link Left_Upper_Leg_Cover: mass 0.4710868540250967 -> 0.075
- link Left_Upper_Leg_Detail: mass 0.0367883220982521 -> 0.01
- link Neck: mass 1.3919244642510382 -> 0.2
- link Rear_Antenna_Box: mass 0.4309225889234217 -> 0.1
- link Rear_Cover: mass 0.4497186658385477 -> 0.15
- link Rear_Head_Plate: mass 0.15477666227232548 -> 0.05
- link Right_Ankle_Cover: mass 0.10517582367621385 -> 0.01
- link Right_Cable_Support: mass 0.4093453218387252 -> 0.08
- link Right_Ear: mass 0.08364474291031353 -> 0.01
- link Right_Eye: mass 0.11621842473165622 -> 0.02
- link Right_Foot: mass 1.8791037124906536 -> 0.22
- link Right_Foot_Cover: mass 0.27789077678038787 -> 0.02
- link Right_Foot_Pad: mass 0.8235307524446847 -> 0.08
- link Right_Front_Cover: mass 0.561072854334117 -> 0.1
- link Right_Head_Support: mass 0.15134820645299715 -> 0.04
- link Right_Hip_Bottom_Holder: mass 0.44482107671145044 -> 0.075
- link Right_Hip_Pitch_Motor: mass 0.880 -> 0.920
- link Right_Hip_Roll_Connector: mass 0.28535016693976095 -> 0.1
- link Right_Hip_Roll_Motor: mass 0.880 -> 0.920
- link Right_Hip_Top_Holder: mass 0.6080984706410996 -> 0.08
- link Right_Hip_Yaw_Motor: mass 0.880 -> 0.920
- link Right_Hip_Yaw_Support: mass 0.8252087483097528 -> 0.08
- link Right_Holder: mass 0.3779808137618351 -> 0.08
- link Right_Knee_Motor: mass 0.880 -> 0.920
- link Right_Lower_Leg: mass 2.86490129434894 -> 0.33
- link Right_Lower_Leg_Cover: mass 0.36564522610609057 -> 0.057
- link Right_Top_Cover: mass 0.3062644628817641 -> 0.03
- link Right_Upper_Leg: mass 4.188552131228702 -> 0.5
- link Right_Upper_Leg_Cover: mass 0.47108685403507133 -> 0.075
- link Right_Upper_Leg_Detail: mass 0.036788321506523086 -> 0.01
- link Top_Base_Frame: mass 0.8850450859385088 -> 0.15
- link base_link: mass 0.6 -> 1
- link imu: mass 0.14185490318820562 -> 0.05
- link imu_mount: mass 0.2546845134769666 -> 0.03

Commit message: update urdf for correct inertias and origin

File: BDX-R-Description/urdf/URDF.urdf (robot description, URDF)
Before this commit: robot URDF, 77 links, 76 joints
Links:
- removed link Front_Grill
- removed link Head_Rear_Cover
- removed link Right_Lower_Leg_Cover
- added link Left_Ear_Holder, mass 0.039089198133902825; collision mesh filename=package://URDF_description/meshes/Left_Ear_Holder.stl scale=0.001 0.001 0.001; visual mesh filename=package://URDF_description/meshes/Left_Ear_Holder.stl scale=0.001 0.001 0.001
- added link Left_Ear_Motor, mass 0.21407639017138763; collision mesh filename=package://URDF_description/meshes/Left_Ear_Motor.stl scale=0.001 0.001 0.001; visual mesh filename=package://URDF_description/meshes/Left_Ear_Motor.stl scale=0.001 0.001 0.001
- added link Orin_Nano_Case, mass 0.5; collision mesh filename=package://URDF_description/meshes/Orin_Nano_Case.stl scale=0.001 0.001 0.001; visual mesh filename=package://URDF_description/meshes/Orin_Nano_Case.stl scale=0.001 0.001 0.001
- added link Rear_Head_Cover, mass 0.3; collision mesh filename=package://URDF_description/meshes/Rear_Head_Cover.stl scale=0.001 0.001 0.001; visual mesh filename=package://URDF_description/meshes/Rear_Head_Cover.stl scale=0.001 0.001 0.001
- added link Right_Ear_Holder, mass 0.039089198133902665; collision mesh filename=package://URDF_description/meshes/Right_Ear_Holder.stl scale=0.001 0.001 0.001; visual mesh filename=package://URDF_description/meshes/Right_Ear_Holder.stl scale=0.001 0.001 0.001
- added link Right_Ear_Motor, mass 0.21407640350583973; collision mesh filename=package://URDF_description/meshes/Right_Ear_Motor.stl scale=0.001 0.001 0.001; visual mesh filename=package://URDF_description/meshes/Right_Ear_Motor.stl scale=0.001 0.001 0.001
- added link Right_Lower_leg-Cover, mass 0.04937375027674599; collision mesh filename=package://URDF_description/meshes/Right_Lower_leg-Cover.stl scale=0.001 0.001 0.001; visual mesh filename=package://URDF_description/meshes/Right_Lower_leg-Cover.stl scale=0.001 0.001 0.001
- link Back_Support: mass 0.1 -> 0.19818519083453695
- link Base_Top_Clamp: mass 0.044 -> 0.04628859676338927
- link Battery: mass 1.25 -> 1.073094288437329
- link Battery_Holder: mass 0.18 -> 0.16209189271424795
- link Camera_Mount: mass 0.04 -> 0.032111017172493185
- link Face: mass 0.1 -> 0.036547681364044626
- link Front_Cover: mass 0.2 -> 0.319189974357708
- link Front_Support: mass 0.15 -> 0.18424409661297098
- link Head_Base_Plate: mass 0.24 -> 0.24167712099257307
- link Head_Pitch_Motor: mass 0.242 -> 0.21407641363122526
- link Head_Pitch_Motor_Support: mass 0.08 -> 0.04464301349288608
- link Head_Roll_Connector: mass 0.05 -> 0.02623495760996857
- link Head_Roll_Motor: mass 0.242 -> 0.21407532118731826
- link Head_Roll_Motor_Mount: mass 0.08 -> 0.06069341482294389
- link Head_Yaw_Motor: mass 0.242 -> 0.214075321187319
- link Left_Ankle_Cover: mass 0.01 -> 0.014202085744813586
- link Left_Ankle_Motor: mass 0.405 -> 0.43362988206706554
- link Left_Cable_Support: mass 0.08 -> 0.05527465492344571
- link Left_Ear: mass 0.01 -> 0.0173058023178019
- link Left_Eye: mass 0.02 -> 0.010759900541269532
- link Left_Foot: mass 0.22 -> 0.253738845261166
- link Left_Foot_Cover: mass 0.02 -> 0.03752369551950594
- link Left_Foot_Pad: mass 0.08 -> 0.11120287867405936
- link Left_Front_Cover: mass 0.1 -> 0.05247574794931451
- link Left_Head_Support: mass 0.04 -> 0.020436827848287157
- link Left_Hip_Bottom_Holder: mass 0.075 -> 0.06006501163237421
- link Left_Hip_Pitch_Motor: mass 0.920 -> 0.9104515289190356
- link Left_Hip_Roll_Connector: mass 0.1 -> 0.09814593711615145
- link Left_Hip_Roll_Motor: mass 0.920 -> 0.9069870657157226
- link Left_Hip_Top_Holder: mass 0.08 -> 0.08211265972988092
- link Left_Hip_Yaw_Motor: mass 0.920 -> 0.9104438184229293
- link Left_Hip_Yaw_Support: mass 0.08 -> 0.10788076345385224
- link Left_Holder: mass 0.08 -> 0.03609216827781493
- link Left_Knee_Motor: mass 0.920 -> 0.9104515217073631
- link Left_Lower_Leg: mass 0.33 -> 0.3868529143335189
- link Left_Lower_Leg_Cover: mass 0.057 -> 0.09180221523312034
- link Left_Top_Cover: mass 0.03 -> 0.02926093594411759
- link Left_Upper_Leg: mass 0.5 -> 0.5655536567558276
- link Left_Upper_Leg_Cover: mass 0.075 -> 0.0636117280594398
- link Left_Upper_Leg_Detail: mass 0.01 -> 0.004967595085878627
- link Neck_Motor: mass 0.405 -> 0.42940231867124456
- link Rear_Antenna_Box: mass 0.1 -> 0.04117094798631419
- link Rear_Cover: mass 0.15 -> 0.31819716922538754
- link Rear_Head_Plate: mass 0.05 -> 0.014787579197992883
- link Right_Ankle_Cover: mass 0.01 -> 0.014202085744813589
- link Right_Ankle_Motor: mass 0.405 -> 0.43363012395690076
- link Right_Cable_Support: mass 0.08 -> 0.055274654923445694
- link Right_Ear: mass 0.01 -> 0.017330282593122717
- link Right_Eye: mass 0.02 -> 0.011103671152706012
- link Right_Foot: mass 0.22 -> 0.25373884525351503
- link Right_Foot_Cover: mass 0.02 -> 0.037524104890090594
- link Right_Foot_Pad: mass 0.08 -> 0.11120287867405933
- link Right_Front_Cover: mass 0.1 -> 0.053605686719820106
- link Right_Head_Support: mass 0.04 -> 0.020436827877729553
- link Right_Hip_Bottom_Holder: mass 0.075 -> 0.060065011632374196
- link Right_Hip_Pitch_Motor: mass 0.920 -> 0.9104438192734086
- link Right_Hip_Roll_Connector: mass 0.1 -> 0.09814591729138275
- link Right_Hip_Roll_Motor: mass 0.920 -> 0.9069872059005614
- link Right_Hip_Top_Holder: mass 0.08 -> 0.08211265972988097
- link Right_Hip_Yaw_Motor: mass 0.920 -> 0.9104438183269751
- link Right_Hip_Yaw_Support: mass 0.08 -> 0.11096680121360432
- link Right_Holder: mass 0.08 -> 0.03611281660144922
- link Right_Knee_Motor: mass 0.920 -> 0.9104438184284508
- link Right_Lower_Leg: mass 0.33 -> 0.38685291363183144
- link Right_Top_Cover: mass 0.03 -> 0.029260935944117595
- link Right_Upper_Leg: mass 0.5 -> 0.5655879310958503
- link Right_Upper_Leg_Cover: mass 0.075 -> 0.0636117280607867
- link Right_Upper_Leg_Detail: mass 0.01 -> 0.004967595005976366
- link Top_Base_Frame: mass 0.15 -> 0.1195092727509324
- link base_link: mass 1 -> 1.1588690647920126
- link imu: mass 0.05 -> 0.1
- link imu_mount: mass 0.03 -> 0.05
Joints:
- removed joint Rigid 37
- removed joint Rigid 38
- removed joint Rigid 39
- removed joint Rigid 40
- removed joint Rigid 58
- added joint Rigid 80: type fixed, parent Front_Support, child Orin_Nano_Case, origin xyz=0.01 -0.02 0.0 rpy=0 0 0
- added joint Rigid 81: type fixed, parent Head_Base_Plate, child Right_Ear_Holder, origin xyz=-0.142593 -0.04359 0.0 rpy=0 0 0
- added joint Rigid 82: type fixed, parent Right_Ear_Holder, child Right_Ear_Motor, origin xyz=-0.021543 0.004139 0.045321 rpy=0 0 0
- added joint Rigid 83: type fixed, parent Right_Ear_Motor, child Right_Ear, origin xyz=0.000669 0.0 -0.019584 rpy=0 0 0
- added joint Rigid 84: type fixed, parent Head_Base_Plate, child Left_Ear_Holder, origin xyz=-0.142593 0.067109 0.0 rpy=0 0 0
- added joint Rigid 85: type fixed, parent Left_Ear_Holder, child Left_Ear_Motor, origin xyz=-0.01245 0.024261 0.032311 rpy=0 0 0
- added joint Rigid 86: type fixed, parent Left_Ear_Motor, child Left_Ear, origin xyz=-0.012545 0.0 0.004702 rpy=0 0 0
- added joint Rigid 87: type fixed, parent Left_Head_Support, child Rear_Head_Cover, origin xyz=-0.008598 -0.001727 0.010956 rpy=0 0 0
- added joint Rigid 88: type fixed, parent Rear_Head_Cover, child Rear_Head_Plate, origin xyz=-0.174901 -0.091107 -0.001821 rpy=0 0 0
- joint Head_Pitch: limit lower=-1.0471975511965976 upper=0.8726646259971648 effort=6.0 velocity=45.0 -> lower=-1.0471975511965976 upper=0.5235987755982988 effort=6.0 velocity=45.0
- joint Left_Knee: origin xyz=0.045459 -0.0025 0.01829 rpy=0 0 0 -> xyz=0.045459 -0.0025 0.018291 rpy=0 0 0
- joint Right_Knee: origin xyz=0.01829 0.0025 -0.045459 rpy=0 0 0 -> xyz=0.01829 0.0025 -0.045458 rpy=0 0 0
- joint Rigid 10: origin xyz=-0.045104 0.01775 0.002892 rpy=0 0 0 -> xyz=0.070648 0.0178 0.088154 rpy=0 0 0
- joint Rigid 11: origin xyz=-0.157 -0.06 0.063636 rpy=0 0 0 -> xyz=-0.041248 -0.05995 0.148898 rpy=0 0 0
- joint Rigid 13: origin xyz=-0.1581 0.090997 0.065042 rpy=0 0 0 -> xyz=-0.042349 0.091047 0.150304 rpy=0 0 0
- joint Rigid 14: origin xyz=-0.148285 0.084346 0.090657 rpy=0 0 0 -> xyz=-0.032533 0.084396 0.175919 rpy=0 0 0
- joint Rigid 16: origin xyz=-0.017969 0.027051 0.074357 rpy=0 0 0 -> xyz=-0.017969 0.027051 0.074557 rpy=0 0 0
- joint Rigid 20: origin xyz=-0.0112 0.01 -0.005406 rpy=0 0 0 -> xyz=0.104552 0.01005 0.079856 rpy=0 0 0
- joint Rigid 23: origin xyz=0.058599 -0.056479 0.0 rpy=0 0 0 -> xyz=0.058598 -0.056479 0.0 rpy=0 0 0
- joint Rigid 24: origin xyz=0.004894 -0.112243 -0.028497 rpy=0 0 0 -> xyz=0.004894 -0.112243 -0.028496 rpy=0 0 0
- joint Rigid 26: origin xyz=0.087134 -0.028034 0.010956 rpy=0 0 0 -> xyz=0.202885 -0.027984 0.096418 rpy=0 0 0
- joint Rigid 27: origin xyz=0.058599 0.109997 0.0 rpy=0 0 0 -> xyz=0.058598 0.109997 0.0 rpy=0 0 0
- joint Rigid 28: origin xyz=-0.1581 -0.090997 0.065042 rpy=0 0 0 -> xyz=-0.042349 -0.090947 0.150304 rpy=0 0 0
- joint Rigid 29: origin xyz=-0.027746 0.157732 0.0 rpy=0 0 0 -> xyz=-0.027747 0.157732 0.0 rpy=0 0 0
- joint Rigid 31: origin xyz=-0.157777 0.0 -0.083128 rpy=0 0 0 -> xyz=-0.042025 5e-05 0.002134 rpy=0 0 0
- joint Rigid 33: origin xyz=-0.024139 -0.0278 0.14533 rpy=0 0 0 -> xyz=0.091613 -0.02775 0.230592 rpy=0 0 0
- joint Rigid 36: origin xyz=0.052962 -0.098148 0.0 rpy=0 0 0 -> xyz=0.052961 -0.098148 0.0 rpy=0 0 0
- joint Rigid 4: origin xyz=-0.148374 0.068751 0.024336 rpy=0 0 0 -> xyz=-0.032622 0.068801 0.109598 rpy=0 0 0
- joint Rigid 49: origin xyz=0.072419 -0.045377 -0.097578 rpy=0 0 0 -> xyz=0.072419 -0.045377 -0.097579 rpy=0 0 0
- joint Rigid 5: origin xyz=-0.148374 -0.068751 0.024336 rpy=0 0 0 -> xyz=-0.032622 -0.068701 0.109598 rpy=0 0 0
- joint Rigid 50: origin xyz=0.009131 -0.00934 -0.124165 rpy=0 0 0 -> xyz=0.009131 -0.00934 -0.124166 rpy=0 0 0
- joint Rigid 52: origin xyz=0.10668 -0.025682 -0.057538 rpy=0 0 0 -> xyz=0.222432 -0.025632 0.027724 rpy=0 0 0
- joint Rigid 54: origin xyz=0.058902 0.0465 -0.075069 rpy=0 0 0 -> xyz=0.058901 0.0465 -0.075069 rpy=0 0 0
- joint Rigid 55: origin xyz=-0.10624 0.0465 -0.111941 rpy=0 0 0 -> xyz=-0.10624 0.0465 -0.11194 rpy=0 0 0
- joint Rigid 56: origin xyz=-0.093612 0.011824 0.044456 rpy=0 0 0 -> xyz=0.022141 0.011874 0.129718 rpy=0 0 0
- joint Rigid 57: origin xyz=0.061778 0.154093 0.101024 rpy=0 0 0 -> xyz=0.177343 0.156643 0.186285 rpy=0 0 0
- joint Rigid 6: origin xyz=0.017134 -0.01645 0.044533 rpy=0 0 0 -> xyz=0.132886 -0.0164 0.129795 rpy=0 0 0
- joint Rigid 68: origin xyz=0.044717 0.00934 -0.09358 rpy=0 0 0 -> xyz=0.044717 0.00934 -0.093581 rpy=0 0 0
- joint Rigid 72: origin xyz=0.058902 -0.0465 -0.075069 rpy=0 0 0 -> xyz=0.058901 -0.0465 -0.075069 rpy=0 0 0
- joint Rigid 73: child Right_Lower_Leg_Cover -> Right_Lower_leg-Cover; origin xyz=-0.10624 -0.0465 -0.111941 rpy=0 0 0 -> xyz=-0.10624 -0.0465 -0.11194 rpy=0 0 0
- joint Rigid 74: origin xyz=-0.093612 -0.011824 0.042716 rpy=0 0 0 -> xyz=0.022141 -0.011774 0.127978 rpy=0 0 0
- joint Rigid 75: origin xyz=0.017878 0.045377 -0.162577 rpy=0 0 0 -> xyz=0.017878 0.045377 -0.162578 rpy=0 0 0
- joint Rigid 8: origin xyz=-0.075084 0.063 -0.123908 rpy=0 0 0 -> xyz=0.040668 0.06305 -0.038646 rpy=0 0 0
- joint Rigid 9: origin xyz=-0.045104 -0.01775 0.002892 rpy=0 0 0 -> xyz=0.070648 -0.0177 0.088154 rpy=0 0 0

Commit message: Update new urdf

File: BDX-R-Description/urdf/URDF.urdf (robot description, URDF)
Before this commit: robot URDF, 81 links, 80 joints
Links:
- removed link Right_Lower_leg-Cover
- added link Right_Lower_Leg_Cover, mass 0.04937375027674599; collision mesh filename=package://URDF_description/meshes/Right_Lower_Leg_Cover.stl scale=0.001 0.001 0.001; visual mesh filename=package://URDF_description/meshes/Right_Lower_Leg_Cover.stl scale=0.001 0.001 0.001
Joints:
- joint Rigid 73: child Right_Lower_leg-Cover -> Right_Lower_Leg_Cover
