Commit message: New xml files

File: BDX-R-Description/urdf/URDF.urdf (robot description, URDF)
Before this commit: robot URDF, 81 links, 80 joints
Links:
- link Back_Support: geometry collision mesh filename=meshes/Back_Support.stl scale=0.001 0.001 0.001; visual mesh filename=meshes/Back_Support.stl scale=0.001 0.001 0.001
- link Base_Top_Clamp: geometry collision mesh filename=meshes/Base_Top_Clamp.stl scale=0.001 0.001 0.001; visual mesh filename=meshes/Base_Top_Clamp.stl scale=0.001 0.001 0.001
- link Battery: geometry collision mesh filename=meshes/Battery.stl scale=0.001 0.001 0.001; visual mesh filename=meshes/Battery.stl scale=0.001 0.001 0.001
- link Battery_Holder: geometry collision mesh filename=meshes/Battery_Holder.stl scale=0.001 0.001 0.001; visual mesh filename=meshes/Battery_Holder.stl scale=0.001 0.001 0.001
- link Bottom_Cover: geometry collision mesh filename=meshes/Bottom_Cover.stl scale=0.001 0.001 0.001; visual mesh filename=meshes/Bottom_Cover.stl scale=0.001 0.001 0.001
- link Camera_Mount: geometry collision mesh filename=meshes/Camera_Mount.stl scale=0.001 0.001 0.001; visual mesh filename=meshes/Camera_Mount.stl scale=0.001 0.001 0.001
- link Face: geometry collision mesh filename=meshes/Face.stl scale=0.001 0.001 0.001; visual mesh filename=meshes/Face.stl scale=0.001 0.001 0.001
- link Front_Cover: geometry collision mesh filename=meshes/Front_Cover.stl scale=0.001 0.001 0.001; visual mesh filename=meshes/Front_Cover.stl scale=0.001 0.001 0.001
- link Front_Support: geometry collision mesh filename=meshes/Front_Support.stl scale=0.001 0.001 0.001; visual mesh filename=meshes/Front_Support.stl scale=0.001 0.001 0.001
- link Head_Base_Plate: geometry collision mesh filename=meshes/Head_Base_Plate.stl scale=0.001 0.001 0.001; visual mesh filename=meshes/Head_Base_Plate.stl scale=0.001 0.001 0.001
- link Head_Pitch_Motor: geometry collision mesh filename=meshes/Head_Pitch_Motor.stl scale=0.001 0.001 0.001; visual mesh filename=meshes/Head_Pitch_Motor.stl scale=0.001 0.001 0.001
- link Head_Pitch_Motor_Support: geometry collision mesh filename=meshes/Head_Pitch_Motor_Support.stl scale=0.001 0.001 0.001; visual mesh filename=meshes/Head_Pitch_Motor_Support.stl scale=0.001 0.001 0.001
- link Head_Roll_Connector: geometry collision mesh filename=meshes/Head_Roll_Connector.stl scale=0.001 0.001 0.001; visual mesh filename=meshes/Head_Roll_Connector.stl scale=0.001 0.001 0.001
- link Head_Roll_Motor: geometry collision mesh filename=meshes/Head_Roll_Motor.stl scale=0.001 0.001 0.001; visual mesh filename=meshes/Head_Roll_Motor.stl scale=0.001 0.001 0.001
- link Head_Roll_Motor_Mount: geometry collision mesh filename=meshes/Head_Roll_Motor_Mount.stl scale=0.001 0.001 0.001; visual mesh filename=meshes/Head_Roll_Motor_Mount.stl scale=0.001 0.001 0.001
- link Head_Yaw_Motor: geometry collision mesh filename=meshes/Head_Yaw_Motor.stl scale=0.001 0.001 0.001; visual mesh filename=meshes/Head_Yaw_Motor.stl scale=0.001 0.001 0.001
- link Left_Ankle_Cover: geometry collision mesh filename=meshes/Left_Ankle_Cover.stl scale=0.001 0.001 0.001; visual mesh filename=meshes/Left_Ankle_Cover.stl scale=0.001 0.001 0.001
- link Left_Ankle_Motor: geometry collision mesh filename=meshes/Left_Ankle_Motor.stl scale=0.001 0.001 0.001; visual mesh filename=meshes/Left_Ankle_Motor.stl scale=0.001 0.001 0.001
- link Left_Cable_Support: geometry collision mesh filename=meshes/Left_Cable_Support.stl scale=0.001 0.001 0.001; visual mesh filename=meshes/Left_Cable_Support.stl scale=0.001 0.001 0.001
- link Left_Ear: geometry collision mesh filename=meshes/Left_Ear.stl scale=0.001 0.001 0.001; visual mesh filename=meshes/Left_Ear.stl scale=0.001 0.001 0.001
- link Left_Ear_Holder: geometry collision mesh filename=meshes/Left_Ear_Holder.stl scale=0.001 0.001 0.001; visual mesh filename=meshes/Left_Ear_Holder.stl scale=0.001 0.001 0.001
- link Left_Ear_Motor: geometry collision mesh filename=meshes/Left_Ear_Motor.stl scale=0.001 0.001 0.001; visual mesh filename=meshes/Left_Ear_Motor.stl scale=0.001 0.001 0.001
- link Left_Eye: geometry collision mesh filename=meshes/Left_Eye.stl scale=0.001 0.001 0.001; visual mesh filename=meshes/Left_Eye.stl scale=0.001 0.001 0.001
- link Left_Foot: geometry collision mesh filename=meshes/Left_Foot.stl scale=0.001 0.001 0.001; visual mesh filename=meshes/Left_Foot.stl scale=0.001 0.001 0.001
- link Left_Foot_Cover: geometry collision mesh filename=meshes/Left_Foot_Cover.stl scale=0.001 0.001 0.001; visual mesh filename=meshes/Left_Foot_Cover.stl scale=0.001 0.001 0.001
- link Left_Foot_Pad: geometry collision mesh filename=meshes/Left_Foot_Pad.stl scale=0.001 0.001 0.001; visual mesh filename=meshes/Left_Foot_Pad.stl scale=0.001 0.001 0.001
- link Left_Front_Cover: geometry collision mesh filename=meshes/Left_Front_Cover.stl scale=0.001 0.001 0.001; visual mesh filename=meshes/Left_Front_Cover.stl scale=0.001 0.001 0.001
- link Left_Head_Support: geometry collision mesh filename=meshes/Left_Head_Support.stl scale=0.001 0.001 0.001; visual mesh filename=meshes/Left_Head_Support.stl scale=0.001 0.001 0.001
- link Left_Hip_Bottom_Holder: geometry collision mesh filename=meshes/Left_Hip_Bottom_Holder.stl scale=0.001 0.001 0.001; visual mesh filename=meshes/Left_Hip_Bottom_Holder.stl scale=0.001 0.001 0.001
- link Left_Hip_Pitch_Motor: geometry collision mesh filename=meshes/Left_Hip_Pitch_Motor.stl scale=0.001 0.001 0.001; visual mesh filename=meshes/Left_Hip_Pitch_Motor.stl scale=0.001 0.001 0.001
- link Left_Hip_Roll_Connector: geometry collision mesh filename=meshes/Left_Hip_Roll_Connector.stl scale=0.001 0.001 0.001; visual mesh filename=meshes/Left_Hip_Roll_Connector.stl scale=0.001 0.001 0.001
- link Left_Hip_Roll_Motor: geometry collision mesh filename=meshes/Left_Hip_Roll_Motor.stl scale=0.001 0.001 0.001; visual mesh filename=meshes/Left_Hip_Roll_Motor.stl scale=0.001 0.001 0.001
- link Left_Hip_Top_Holder: geometry collision mesh filename=meshes/Left_Hip_Top_Holder.stl scale=0.001 0.001 0.001; visual mesh filename=meshes/Left_Hip_Top_Holder.stl scale=0.001 0.001 0.001
- link Left_Hip_Yaw_Motor: geometry collision mesh filename=meshes/Left_Hip_Yaw_Motor.stl scale=0.001 0.001 0.001; visual mesh filename=meshes/Left_Hip_Yaw_Motor.stl scale=0.001 0.001 0.001
- link Left_Hip_Yaw_Support: geometry collision mesh filename=meshes/Left_Hip_Yaw_Support.stl scale=0.001 0.001 0.001; visual mesh filename=meshes/Left_Hip_Yaw_Support.stl scale=0.001 0.001 0.001
- link Left_Holder: geometry collision mesh filename=meshes/Left_Holder.stl scale=0.001 0.001 0.001; visual mesh filename=meshes/Left_Holder.stl scale=0.001 0.001 0.001
- link Left_Knee_Motor: geometry collision mesh filename=meshes/Left_Knee_Motor.stl scale=0.001 0.001 0.001; visual mesh filename=meshes/Left_Knee_Motor.stl scale=0.001 0.001 0.001
- link Left_Lower_Leg: geometry collision mesh filename=meshes/Left_Lower_Leg.stl scale=0.001 0.001 0.001; visual mesh filename=meshes/Left_Lower_Leg.stl scale=0.001 0.001 0.001
- link Left_Lower_Leg_Cover: geometry collision mesh filename=meshes/Left_Lower_Leg_Cover.stl scale=0.001 0.001 0.001; visual mesh filename=meshes/Left_Lower_Leg_Cover.stl scale=0.001 0.001 0.001
- link Left_Top_Cover: geometry collision mesh filename=meshes/Left_Top_Cover.stl scale=0.001 0.001 0.001; visual mesh filename=meshes/Left_Top_Cover.stl scale=0.001 0.001 0.001
- link Left_Upper_Leg: geometry collision mesh filename=meshes/Left_Upper_Leg.stl scale=0.001 0.001 0.001; visual mesh filename=meshes/Left_Upper_Leg.stl scale=0.001 0.001 0.001
- link Left_Upper_Leg_Cover: geometry collision mesh filename=meshes/Left_Upper_Leg_Cover.stl scale=0.001 0.001 0.001; visual mesh filename=meshes/Left_Upper_Leg_Cover.stl scale=0.001 0.001 0.001
- link Left_Upper_Leg_Detail: geometry collision mesh filename=meshes/Left_Upper_Leg_Detail.stl scale=0.001 0.001 0.001; visual mesh filename=meshes/Left_Upper_Leg_Detail.stl scale=0.001 0.001 0.001
- link Neck: geometry collision mesh filename=meshes/Neck.stl scale=0.001 0.001 0.001; visual mesh filename=meshes/Neck.stl scale=0.001 0.001 0.001
- link Neck_Motor: geometry collision mesh filename=meshes/Neck_Motor.stl scale=0.001 0.001 0.001; visual mesh filename=meshes/Neck_Motor.stl scale=0.001 0.001 0.001
- link Orin_Nano_Case: geometry collision mesh filename=meshes/Orin_Nano_Case.stl scale=0.001 0.001 0.001; visual mesh filename=meshes/Orin_Nano_Case.stl scale=0.001 0.001 0.001
- link Rear_Antenna_Box: geometry collision mesh filename=meshes/Rear_Antenna_Box.stl scale=0.001 0.001 0.001; visual mesh filename=meshes/Rear_Antenna_Box.stl scale=0.001 0.001 0.001
- link Rear_Cover: geometry collision mesh filename=meshes/Rear_Cover.stl scale=0.001 0.001 0.001; visual mesh filename=meshes/Rear_Cover.stl scale=0.001 0.001 0.001
- link Rear_Head_Cover: geometry collision mesh filename=meshes/Rear_Head_Cover.stl scale=0.001 0.001 0.001; visual mesh filename=meshes/Rear_Head_Cover.stl scale=0.001 0.001 0.001
- link Rear_Head_Plate: geometry collision mesh filename=meshes/Rear_Head_Plate.stl scale=0.001 0.001 0.001; visual mesh filename=meshes/Rear_Head_Plate.stl scale=0.001 0.001 0.001
- link Right_Ankle_Cover: geometry collision mesh filename=meshes/Right_Ankle_Cover.stl scale=0.001 0.001 0.001; visual mesh filename=meshes/Right_Ankle_Cover.stl scale=0.001 0.001 0.001
- link Right_Ankle_Motor: geometry collision mesh filename=meshes/Right_Ankle_Motor.stl scale=0.001 0.001 0.001; visual mesh filename=meshes/Right_Ankle_Motor.stl scale=0.001 0.001 0.001
- link Right_Cable_Support: geometry collision mesh filename=meshes/Right_Cable_Support.stl scale=0.001 0.001 0.001; visual mesh filename=meshes/Right_Cable_Support.stl scale=0.001 0.001 0.001
- link Right_Ear: geometry collision mesh filename=meshes/Right_Ear.stl scale=0.001 0.001 0.001; visual mesh filename=meshes/Right_Ear.stl scale=0.001 0.001 0.001
- link Right_Ear_Holder: geometry collision mesh filename=meshes/Right_Ear_Holder.stl scale=0.001 0.001 0.001; visual mesh filename=meshes/Right_Ear_Holder.stl scale=0.001 0.001 0.001
- link Right_Ear_Motor: geometry collision mesh filename=meshes/Right_Ear_Motor.stl scale=0.001 0.001 0.001; visual mesh filename=meshes/Right_Ear_Motor.stl scale=0.001 0.001 0.001
- link Right_Eye: geometry collision mesh filename=meshes/Right_Eye.stl scale=0.001 0.001 0.001; visual mesh filename=meshes/Right_Eye.stl scale=0.001 0.001 0.001
- link Right_Foot: geometry collision mesh filename=meshes/Right_Foot.stl scale=0.001 0.001 0.001; visual mesh filename=meshes/Right_Foot.stl scale=0.001 0.001 0.001
- link Right_Foot_Cover: geometry collision mesh filename=meshes/Right_Foot_Cover.stl scale=0.001 0.001 0.001; visual mesh filename=meshes/Right_Foot_Cover.stl scale=0.001 0.001 0.001
- link Right_Foot_Pad: geometry collision mesh filename=meshes/Right_Foot_Pad.stl scale=0.001 0.001 0.001; visual mesh filename=meshes/Right_Foot_Pad.stl scale=0.001 0.001 0.001
- link Right_Front_Cover: geometry collision mesh filename=meshes/Right_Front_Cover.stl scale=0.001 0.001 0.001; visual mesh filename=meshes/Right_Front_Cover.stl scale=0.001 0.001 0.001
- link Right_Head_Support: geometry collision mesh filename=meshes/Right_Head_Support.stl scale=0.001 0.001 0.001; visual mesh filename=meshes/Right_Head_Support.stl scale=0.001 0.001 0.001
- link Right_Hip_Bottom_Holder: geometry collision mesh filename=meshes/Right_Hip_Bottom_Holder.stl scale=0.001 0.001 0.001; visual mesh filename=meshes/Right_Hip_Bottom_Holder.stl scale=0.001 0.001 0.001
- link Right_Hip_Pitch_Motor: geometry collision mesh filename=meshes/Right_Hip_Pitch_Motor.stl scale=0.001 0.001 0.001; visual mesh filename=meshes/Right_Hip_Pitch_Motor.stl scale=0.001 0.001 0.001
- link Right_Hip_Roll_Connector: geometry collision mesh filename=meshes/Right_Hip_Roll_Connector.stl scale=0.001 0.001 0.001; visual mesh filename=meshes/Right_Hip_Roll_Connector.stl scale=0.001 0.001 0.001
- link Right_Hip_Roll_Motor: geometry collision mesh filename=meshes/Right_Hip_Roll_Motor.stl scale=0.001 0.001 0.001; visual mesh filename=meshes/Right_Hip_Roll_Motor.stl scale=0.001 0.001 0.001
- link Right_Hip_Top_Holder: geometry collision mesh filename=meshes/Right_Hip_Top_Holder.stl scale=0.001 0.001 0.001; visual mesh filename=meshes/Right_Hip_Top_Holder.stl scale=0.001 0.001 0.001
- link Right_Hip_Yaw_Motor: geometry collision mesh filename=meshes/Right_Hip_Yaw_Motor.stl scale=0.001 0.001 0.001; visual mesh filename=meshes/Right_Hip_Yaw_Motor.stl scale=0.001 0.001 0.001
- link Right_Hip_Yaw_Support: geometry collision mesh filename=meshes/Right_Hip_Yaw_Support.stl scale=0.001 0.001 0.001; visual mesh filename=meshes/Right_Hip_Yaw_Support.stl scale=0.001 0.001 0.001
- link Right_Holder: geometry collision mesh filename=meshes/Right_Holder.stl scale=0.001 0.001 0.001; visual mesh filename=meshes/Right_Holder.stl scale=0.001 0.001 0.001
- link Right_Knee_Motor: geometry collision mesh filename=meshes/Right_Knee_Motor.stl scale=0.001 0.001 0.001; visual mesh filename=meshes/Right_Knee_Motor.stl scale=0.001 0.001 0.001
- link Right_Lower_Leg: geometry collision mesh filename=meshes/Right_Lower_Leg.stl scale=0.001 0.001 0.001; visual mesh filename=meshes/Right_Lower_Leg.stl scale=0.001 0.001 0.001
- link Right_Lower_Leg_Cover: geometry collision mesh filename=meshes/Right_Lower_Leg_Cover.stl scale=0.001 0.001 0.001; visual mesh filename=meshes/Right_Lower_Leg_Cover.stl scale=0.001 0.001 0.001
- link Right_Top_Cover: geometry collision mesh filename=meshes/Right_Top_Cover.stl scale=0.001 0.001 0.001; visual mesh filename=meshes/Right_Top_Cover.stl scale=0.001 0.001 0.001
- link Right_Upper_Leg: geometry collision mesh filename=meshes/Right_Upper_Leg.stl scale=0.001 0.001 0.001; visual mesh filename=meshes/Right_Upper_Leg.stl scale=0.001 0.001 0.001
- link Right_Upper_Leg_Cover: geometry collision mesh filename=meshes/Right_Upper_Leg_Cover.stl scale=0.001 0.001 0.001; visual mesh filename=meshes/Right_Upper_Leg_Cover.stl scale=0.001 0.001 0.001
- link Right_Upper_Leg_Detail: geometry collision mesh filename=meshes/Right_Upper_Leg_Detail.stl scale=0.001 0.001 0.001; visual mesh filename=meshes/Right_Upper_Leg_Detail.stl scale=0.001 0.001 0.001
- link Top_Base_Frame: geometry collision mesh filename=meshes/Top_Base_Frame.stl scale=0.001 0.001 0.001; visual mesh filename=meshes/Top_Base_Frame.stl scale=0.001 0.001 0.001
- link base_link: geometry collision mesh filename=meshes/base_link.stl scale=0.001 0.001 0.001; visual mesh filename=meshes/base_link.stl scale=0.001 0.001 0.001
- link imu: geometry collision mesh filename=meshes/imu.stl scale=0.001 0.001 0.001; visual mesh filename=meshes/imu.stl scale=0.001 0.001 0.001
- link imu_mount: geometry collision mesh filename=meshes/imu_mount.stl scale=0.001 0.001 0.001; visual mesh filename=meshes/imu_mount.stl scale=0.001 0.001 0.001
